File: eagle/808sn.brd (EAGLE design)
At the start: 100 x 80 mm, 82 parts, among them IC1 TL072P, IC3 TL072P, Q1 2N3904, Q45 2N3904, Q46 2N3906, Q47 2N3904, Q48 2N3904, Q49 2N3904

Commit message: 92pct autorouted
Parts:
- R203: device TR808clone:0207/5V -> TR808clone:0309/10
- moved R193 21.7 mm to (10.2, 62.2)
- moved R194 21.6 mm to (6.35, 57.1)
- moved Q48 20.5 mm to (10.2, 47.0)
- moved OUTPUT_NORM 16.6 mm to (73.7, 14.0), turned to 270 degrees
- moved R185 11.7 mm to (19.1, 62.2)
- moved D54 10.9 mm to (24.1, 68.6)
- moved C54 10.5 mm to (30.5, 64.8), turned to 0 degrees
- moved C55 10.2 mm to (26.7, 19.1), turned to 0 degrees
- moved R128 9.25 mm to (30.5, 53.3)
- moved C53 9.16 mm to (21.6, 73.7)
- moved R186 8.52 mm to (19.1, 20.3), turned to 180 degrees
- moved C29 8.52 mm to (24.1, 61.0), turned to 90 degrees
- moved C52 7.73 mm to (15.2, 59.7)
- moved R184 7.41 mm to (16.5, 48.3), turned to 90 degrees
- moved C1 7.18 mm to (24.1, 36.8)
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
Commit message: board started over
Parts:
- C52: device TR808clone:C075-032X103 -> TR808clone:C050-045X075
- C6: device TR808clone:C025-025X050 -> TR808clone:C050-025X075
- C69: device TR808clone:C035-025X75 -> TR808clone:C075-042X103
- R194, R203: device TR808clone:0309/10 -> TR808clone:0207/7
- R204: device TR808clone:0207/5V -> TR808clone:0207/7
- moved OUTPUT 74.9 mm to (15.2, 0.00)
- moved TM4 74.3 mm to (14.0, 62.2)
- moved R130 71.1 mm to (20.3, 61.0), turned to 90 degrees
- moved OUTPUT_NORM 68.1 mm to (6.35, 24.1), turned to 180 degrees
- moved R190 66.1 mm to (94.0, 40.6), turned to 180 degrees
- moved R129 64.3 mm to (21.6, 50.8)
- moved C31 59.8 mm to (7.62, 55.9), turned to 270 degrees
- moved IC3 58.3 mm to (15.2, 44.5), turned to 180 degrees
- moved R131 57.2 mm to (11.4, 52.1)
- moved R189 56.6 mm to (88.9, 31.8)
- moved R207 55.9 mm to (19.1, 19.1), turned to 180 degrees
- moved R193 55.8 mm to (52.1, 25.4), turned to 0 degrees
- moved C57 55.3 mm to (87.6, 35.6), turned to 0 degrees
- moved R206 54.6 mm to (8.89, 36.8)
- moved C52 48.6 mm to (41.9, 19.1), turned to 270 degrees
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Connections:
- net N$30: now also C69.1; no longer C69.P$1
- net N$36: now also C69.2; no longer C69.P$2

Commit message: 94pct autorouted
Parts:
- R183, R189: device TR808clone:0207/5V -> TR808clone:0207/2V
- R186: device TR808clone:0207/5V -> TR808clone:0309/12
- moved C68 17.8 mm to (25.4, 16.5)
- moved GATE 12.5 mm to (76.2, 53.3)
- moved R186 11.5 mm to (62.2, 22.9)
- moved R180 10.5 mm to (81.3, 55.9), turned to 180 degrees
- moved R196 8.03 mm to (91.4, 26.7), turned to 180 degrees
- moved Q47 8.03 mm to (61.0, 34.3), turned to 180 degrees
- moved C51 7.62 mm to (48.3, 41.9)
- moved R190 6.84 mm to (91.4, 34.3), turned to 270 degrees
- moved Q48 6.48 mm to (33.0, 48.3), turned to 90 degrees
- moved R124 6.35 mm to (29.2, 61.0), turned to 0 degrees
- moved C56 5.68 mm to (25.4, 50.8)
- moved R182 5.68 mm to (91.4, 47.0)
- moved C54 5.68 mm to (41.9, 48.3)
- moved TM4 5.39 mm to (17.8, 66.0)
- moved R189 5.39 mm to (85.1, 27.9), turned to 270 degrees
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
Commit message: routed
Parts:
- C31: device TR808clone:E2,5-5 -> TR808clone:E3,5-8
- C51: device TR808clone:E2-5 -> TR808clone:E3,5-8
- R184, R185: device TR808clone:0207/5V -> TR808clone:0207/7
- R189: device TR808clone:0207/2V -> TR808clone:0207/5V
- moved ACCENT 13.5 mm to (71.1, 53.3)
- moved R198 13.3 mm to (54.1, 21.6), turned to 270 degrees
- moved R201 9.67 mm to (29.2, 27.9)
- moved R203 9.25 mm to (30.5, 25.4)
- moved R190 5.18 mm to (90.4, 39.4), turned to 180 degrees
- moved U$1 5.11 mm to (66.3, 48.8)
- moved C57 5.08 mm to (88.9, 34.3)
- moved Q49 5.08 mm to (31.8, 19.1), turned to 0 degrees
- moved PWR1 4.58 mm to (54.6, 61.0)
- moved R205 3.98 mm to (12.2, 29.5)
- moved C5 3.88 mm to (61.5, 48.8)
- moved R180 3.78 mm to (77.7, 57.1)
- moved U$2 3.56 mm to (50.8, 48.5)
- moved C7 3.54 mm to (55.9, 48.8)
- moved R196 3.31 mm to (93.2, 29.5), turned to 270 degrees
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Connections:
- net GND: now also C5.-, C7.+, PWR1.3, PWR1.4, PWR1.5, PWR1.6, PWR1.7, PWR1.8
- net N$26: no longer C5.-, C7.+, PWR1.3, PWR1.4, PWR1.5, PWR1.6, PWR1.7, PWR1.8
Routing:
- net GND: track 0.00 -> 469.7 mm, vias 0 -> 2
- net -12V: track 0.00 -> 173.5 mm, vias 0 -> 6
- net +12V: track 0.00 -> 170.7 mm, vias 0 -> 2
- net N$9: track 0.00 -> 56.2 mm
- net N$35: track 0.00 -> 45.7 mm
- net N$17: track 0.00 -> 38.7 mm
- net TRIG: track 0.00 -> 34.7 mm
- net N$129: track 0.00 -> 30.4 mm
- net N$14: track 0.00 -> 25.6 mm
- net WN1: track 0.00 -> 24.0 mm
- net N$34: track 0.00 -> 21.9 mm
- net N$160: track 0.00 -> 21.7 mm
- net N$8: track 0.00 -> 21.3 mm
- net N$26: track 0.00 -> 20.0 mm
- net N$12: track 0.00 -> 17.2 mm
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
Commit message: tweaks
Parts:
- moved C65 10.4 mm to (58.9, 10.7), turned to 0 degrees
- moved C63 10.4 mm to (86.4, 9.14), turned to 270 degrees
- moved SNAPPY 7.88 mm to (75.2, 3.56)
- moved TONE 3.56 mm to (51.8, 3.81)
- moved R202 3.07 mm to (32.5, 37.1)
- moved R188 2.84 mm to (29.2, 41.9), turned to 90 degrees
- moved C4 2.03 mm to (69.8, 18.5)
- moved R182 0.51 mm to (90.4, 47.5)
Routing:
- net GND: track 469.7 -> 462.7 mm
- net N$17: track 38.7 -> 44.4 mm
- net N$20: track 11.8 -> 16.9 mm
- net N$22: track 15.3 -> 19.5 mm
- net N$34: track 21.9 -> 25.4 mm
- net N$12: track 17.2 -> 14.2 mm
- net N$9: track 56.2 -> 53.6 mm
- net N$18: track 10.7 -> 8.31 mm
- net +12V: track 170.7 -> 169.1 mm
- net N$29: track 15.6 -> 14.2 mm
- net N$28: track 8.29 -> 7.30 mm
- net N$35: track 45.7 -> 44.8 mm
- net N$19: track 3.06 -> 2.50 mm

Commit message: tweaks
Parts:
- moved 130MV_RMS_TP 1.27 mm to (5.08, 43.2)
Routing:
- net WN1: track 24.0 -> 22.7 mm
Changed lines of the file:
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@@
 </autorouter>
 <elements>
-<element name="130MV_RMS_TP" library="con-molex" package="22-23-2021" value="22-23-2021" x="3.81" y="43.18" rot="R180">
-<attribute name="OC_NEWARK" value="25C3832" x="3.81" y="43.18" size="1.778" layer="27" rot="R180" display="off"/>
-<attribute name="MPN" value="22-23-2021" x="3.81" y="43.18" size="1.778" layer="27" rot="R180" display="off"/>
-<attribute name="MF" value="MOLEX" x="3.81" y="43.18" size="1.778" layer="27" rot="R180" display="off"/>
-<attribute name="OC_FARNELL" value="1462926" x="3.81" y="43.18" size="1.778" layer="27" rot="R180" display="off"/>
+<element name="130MV_RMS_TP" library="con-molex" package="22-23-2021" value="22-23-2021" x="5.08" y="43.18" rot="R180">
+<attribute name="OC_NEWARK" value="25C3832" x="5.08" y="43.18" size="1.778" layer="27" rot="R180" display="off"/>
+<attribute name="MPN" value="22-23-2021" x="5.08" y="43.18" size="1.778" layer="27" rot="R180" display="off"/>
+<attribute name="MF" value="MOLEX" x="5.08" y="43.18" size="1.778" layer="27" rot="R180" display="off"/>
+<attribute name="OC_FARNELL" value="1462926" x="5.08" y="43.18" size="1.778" layer="27" rot="R180" display="off"/>
 </element>
 <element name="ACCENT" library="solpad" package="LSP10" value="LSP10" x="71.12" y="53.34"/>
@@
 <wire x1="25.5905" y1="65.2145" x2="39.624" y2="65.2145" width="1.016" layer="16"/>
 <wire x1="22.733" y1="70.358" x2="25.5905" y2="65.2145" width="1.016" layer="16"/>
-<wire x1="11.684" y1="70.358" x2="22.733" y2="70.358" width="1.016" layer="16"/>
-<wire x1="9.271" y1="67.945" x2="11.684" y2="70.358" width="1.016" layer="16"/>
+<wire x1="11.43" y1="70.358" x2="22.733" y2="70.358" width="1.016" layer="16"/>
+<wire x1="9.017" y1="67.945" x2="11.43" y2="70.358" width="1.016" layer="16"/>
 <wire x1="39.624" y1="65.2145" x2="40.7035" y2="65.151" width="1.016" layer="16"/>
 <contactref element="C7" pad="+"/>
@@
 <contactref element="R188" pad="1"/>
 <contactref element="C53" pad="P$2"/>
-<wire x1="9.271" y1="67.945" x2="8.89" y2="67.945" width="1.016" layer="16"/>
+<wire x1="9.017" y1="67.945" x2="8.89" y2="67.945" width="1.016" layer="16"/>
 <wire x1="8.89" y1="67.945" x2="7.62" y2="66.675" width="1.016" layer="16"/>
-<wire x1="2.54" y1="43.18" x2="2.286" y2="47.752" width="1.016" layer="16"/>
+<wire x1="3.81" y1="43.18" x2="2.286" y2="47.752" width="1.016" layer="16"/>
 <wire x1="2.286" y1="47.752" x2="6.35" y2="48.26" width="1.016" layer="16"/>
 <wire x1="7.62" y1="66.675" x2="4.445" y2="66.675" width="1.016" layer="16"/>
@@
 <wire x1="3.81" y1="66.04" x2="2.286" y2="60.198" width="1.016" layer="16"/>
 <wire x1="2.286" y1="60.198" x2="2.032" y2="50.8" width="1.016" layer="16"/>
-<wire x1="2.032" y1="50.8" x2="2.54" y2="43.18" width="1.016" layer="16"/>
+<wire x1="2.032" y1="50.8" x2="3.81" y2="43.18" width="1.016" layer="16"/>
 <wire x1="25.4" y1="40.64" x2="26.67" y2="40.64" width="1.016" layer="16"/>
 <wire x1="26.67" y1="40.64" x2="29.21" y2="39.37" width="1.016" layer="16"/>
@@
 <wire x1="6.35" y1="6.39" x2="10.24" y2="2.5" width="1.016" layer="16"/>
 <wire x1="6.35" y1="25.4" x2="5.08" y2="36.83" width="1.016" layer="16"/>
-<wire x1="2.54" y1="43.18" x2="2.54" y2="38.1" width="1.016" layer="16"/>
-<wire x1="2.54" y1="38.1" x2="3.81" y2="36.83" width="1.016" layer="16"/>
+<wire x1="3.81" y1="43.18" x2="3.81" y2="36.83" width="1.016" layer="16"/>
 <wire x1="3.81" y1="36.83" x2="5.08" y2="36.83" width="1.016" layer="16"/>
 <wire x1="93.218" y1="33.274" x2="93.218" y2="39.116" width="1.016" layer="16"/>
@@
 <wire x1="22.86" y1="50.8" x2="23.1775" y2="50.8" width="0.8128" layer="16"/>
 <wire x1="23.1775" y1="50.8" x2="23.4" y2="50.8" width="0.8128" layer="16"/>
-<wire x1="16.8275" y1="44.45" x2="5.08" y2="43.18" width="0.8128" layer="16"/>
+<wire x1="16.8275" y1="44.45" x2="6.35" y2="43.18" width="0.8128" layer="16"/>
 <wire x1="19.05" y1="47.9425" x2="16.8275" y2="44.45" width="0.8128" layer="16"/>
 <wire x1="19.05" y1="47.9425" x2="19.05" y2="48.26" width="0.8128" layer="16"/>

Commit message: cutout
Routing:
- net GND: track 462.6 -> 461.9 mm
Other:
- board size 100 x 80 mm -> 100 x 81.3 mm
Changed lines of the file:
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@@
 <layer number="44" name="Drills" color="7" fill="1" visible="no" active="yes"/>
 <layer number="45" name="Holes" color="7" fill="1" visible="no" active="yes"/>
-<layer number="46" name="Milling" color="3" fill="1" visible="no" active="yes"/>
+<layer number="46" name="Milling" color="3" fill="1" visible="yes" active="yes"/>
 <layer number="47" name="Measures" color="7" fill="1" visible="no" active="yes"/>
 <layer number="48" name="Document" color="7" fill="1" visible="yes" active="yes"/>
@@
 <wire x1="0" y1="80" x2="0" y2="0" width="0" layer="20"/>
 <rectangle x1="50.8" y1="59.69" x2="55.88" y2="62.23" layer="16"/>
+<wire x1="1.27" y1="72.39" x2="95.25" y2="72.39" width="1.6764" layer="46"/>
+<wire x1="95.25" y1="72.39" x2="96.52" y2="71.12" width="1.6764" layer="46"/>
+<wire x1="96.52" y1="71.12" x2="96.52" y2="0" width="1.6764" layer="46"/>
+<wire x1="96.52" y1="0" x2="95.25" y2="-1.27" width="1.6764" layer="46"/>
+<wire x1="95.25" y1="-1.27" x2="1.27" y2="-1.27" width="1.6764" layer="46"/>
+<wire x1="1.27" y1="-1.27" x2="0" y2="0" width="1.6764" layer="46"/>
+<wire x1="0" y1="0" x2="0" y2="71.12" width="1.6764" layer="46"/>
+<wire x1="0" y1="71.12" x2="1.27" y2="72.39" width="1.6764" layer="46"/>
+<wire x1="91.44" y1="68.58" x2="91.44" y2="67.31" width="1.6764" layer="46"/>
+<wire x1="91.44" y1="67.31" x2="92.71" y2="67.31" width="1.6764" layer="46"/>
+<wire x1="92.71" y1="67.31" x2="92.71" y2="68.58" width="1.6764" layer="46"/>
+<wire x1="92.71" y1="68.58" x2="91.44" y2="68.58" width="1.6764" layer="46"/>
+<wire x1="91.44" y1="3.81" x2="91.44" y2="2.54" width="1.6764" layer="46"/>
+<wire x1="91.44" y1="2.54" x2="92.71" y2="2.54" width="1.6764" layer="46"/>
+<wire x1="92.71" y1="2.54" x2="92.71" y2="3.81" width="1.6764" layer="46"/>
+<wire x1="92.71" y1="3.81" x2="91.44" y2="3.81" width="1.6764" layer="46"/>
+<wire x1="3.81" y1="6.35" x2="3.81" y2="5.08" width="1.6764" layer="46"/>
+<wire x1="3.81" y1="5.08" x2="5.08" y2="5.08" width="1.6764" layer="46"/>
+<wire x1="5.08" y1="5.08" x2="5.08" y2="6.35" width="1.6764" layer="46"/>
+<wire x1="5.08" y1="6.35" x2="3.81" y2="6.35" width="1.6764" layer="46"/>
+<wire x1="55.88" y1="43.18" x2="55.88" y2="41.91" width="1.6764" layer="46"/>
+<wire x1="55.88" y1="41.91" x2="57.15" y2="41.91" width="1.6764" layer="46"/>
+<wire x1="57.15" y1="41.91" x2="57.15" y2="43.18" width="1.6764" layer="46"/>
+<wire x1="57.15" y1="43.18" x2="55.88" y2="43.18" width="1.6764" layer="46"/>
 </plain>
 <attributes>
@@
 <wire x1="57.15" y1="17.78" x2="58.42" y2="19.05" width="1.016" layer="16"/>
 <wire x1="68.58" y1="18.542" x2="67.31" y2="18.796" width="1.016" layer="16"/>
-<wire x1="6.35" y1="25.4" x2="6.35" y2="6.39" width="1.016" layer="16"/>
-<wire x1="6.35" y1="6.39" x2="10.24" y2="2.5" width="1.016" layer="16"/>
+<wire x1="6.35" y1="25.4" x2="5.588" y2="14.264" width="1.016" layer="16"/>
+<wire x1="5.588" y1="14.264" x2="10.24" y2="2.5" width="1.016" layer="16"/>
 <wire x1="6.35" y1="25.4" x2="5.08" y2="36.83" width="1.016" layer="16"/>
 <wire x1="3.81" y1="43.18" x2="3.81" y2="36.83" width="1.016" layer="16"/>
